File: Cloudnine_rp2040.kicad_pcb (KiCad board)
At the start: 2 copper layers, 284.2 x 94.7 mm, 163 parts, among them J2 Conn_01x04, U1 RP2040, U2 XC6206PxxxMR, U3 W25Q128JVS, U4 SRV05-4, Y1 ABM8-272-T3

Commit message: V1.0
Parts:
- added REF**: Stabilizer_MX_2.00u_Slikscreen, ScottoKeebs_Stabilizer:Stabilizer_MX_2.00u_Slikscreen, F.Cu at (280.2, 90.2)
- moved BOOTSEL1 7.38 mm to (98.8, 107.7), turned to -90 degrees
- moved R3 3.82 mm to (36.3, 79.0), turned to 180 degrees
Connections:
- D65 pad 1: GND -> Net-(D65-K)
- D65 pad 2: Net-(D65-A) -> GND
- R3 pad 1: Net-(D65-A) -> Net-(D65-K)
- U1 pad 11: unconnected-(U1-GPIO8-Pad11) -> Row0
- U1 pad 12: unconnected-(U1-GPIO9-Pad12) -> Row1
- U1 pad 13: unconnected-(U1-GPIO10-Pad13) -> Row2
- U1 pad 2: unconnected-(U1-GPIO0-Pad2) -> Row4
- U1 pad 7: unconnected-(U1-GPIO5-Pad7) -> Row3
Routing:
- net unconnected-(U1-GPIO8-Pad11): track 83.7 -> 0.00 mm, vias 1 -> 0
- net Row0: track 268.7 -> 350.5 mm, vias 0 -> 2
- net Row1: track 260.8 -> 316.6 mm, vias 0 -> 2
- net unconnected-(U1-GPIO9-Pad12): track 55.2 -> 0.00 mm, vias 1 -> 0
- net Row4: track 257.0 -> 302.7 mm
- net unconnected-(U1-GPIO0-Pad2): track 39.3 -> 0.00 mm
- net unconnected-(U1-GPIO10-Pad13): track 36.0 -> 0.00 mm, vias 1 -> 0
- net Row2: track 233.9 -> 269.9 mm, vias 0 -> 2
- net Row3: track 254.1 -> 281.9 mm
- net unconnected-(U1-GPIO5-Pad7): track 26.0 -> 0.00 mm
- net Net-(D65-A): track 11.0 -> 0.00 mm
- net Col11: track 228.8 -> 238.3 mm
- net Net-(D54-A): track 7.36 -> 16.9 mm
- net Net-(BOOTSEL1-Pad2): track 7.90 -> 16.3 mm
- net GND: track 2.28 -> 10.7 mm, vias 15 -> 83
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
Commit message: V1.1
Parts:
- moved MX5 0.58 mm to (106.9, 33.2)
- moved D5 0.58 mm to (115.0, 35.8)
Routing:
- net Row0: track 350.5 -> 351.2 mm

Commit message: V1.2
홀 크기 조정
Parts:
- MX1, MX10, MX11, MX12, MX13, MX14, MX15, MX16, MX17, MX18, MX19, MX2, MX20, MX21, MX22, MX23, MX24, MX25, MX26, MX27, MX28, MX29, MX3, MX30, MX31, MX32, MX33, MX34, MX35, MX36, MX37, MX38, MX39, MX4, MX40, MX41, MX42, MX43, MX44, MX45, MX46, MX47, MX48, MX49, MX5, MX50, MX51, MX52, MX53, MX54, MX55, MX56, MX57, MX58, MX59, MX6, MX60, MX61, MX62, MX63, MX7, MX8, MX9: footprint ScottoKeebs_MX:MX_PCB_1.00u_NoSilkscreen3 -> ScottoKeebs_MX:MX_PCB_1.00u_NoSilkscreen_narrow
