File: Cloudnine_rp2040.kicad_sch (KiCad schematic)
At the start: 157 parts, among them J2 Conn_01x04, U1 RP2040, U2 XC6206PxxxMR, U3 W25Q128JVS, U4 SRV05-4, Y1 ABM8-272-T3

Commit message: V1.2
홀 크기 조정
Parts:
- MX1, MX10, MX11, MX12, MX13, MX14, MX15, MX16, MX17, MX18, MX19, MX2, MX20, MX21, MX22, MX23, MX24, MX25, MX26, MX27, MX28, MX29, MX3, MX30, MX31, MX32, MX33, MX34, MX35, MX36, MX37, MX38, MX39, MX4, MX40, MX41, MX42, MX43, MX44, MX45, MX46, MX47, MX48, MX49, MX5, MX50, MX51, MX52, MX53, MX54, MX55, MX56, MX57, MX58, MX59, MX6, MX60, MX61, MX62, MX63, MX7, MX8, MX9: footprint ScottoKeebs_MX:MX_PCB_1.00u_NoSilkscreen3 -> ScottoKeebs_MX:MX_PCB_1.00u_NoSilkscreen_narrow
